File: circuitAndPowerStruct/circuitAndPowerStruct.kicad_sch (KiCad schematic)
At the start: 1 part

Commit message: idk
Other:
- note added: "Estop under voltage"
Changed lines of the file:
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@@
+	)
+	(rectangle
+		(start 204.978 36.322)
+		(end 223.52 45.72)
+		(stroke
+			(width 0)
+			(type default)
+		)
+		(fill
+			(type none)
+		)
 	)
 	(rectangle
@@
 		(exclude_from_sim no)
 		(at 88.265 95.885 0)
+		(effects
+			(font
+				(size 1.27 1.27)
+			)
+		)
+	)
+	(text "Estop \nunder voltage\n"
+		(exclude_from_sim no)
+		(at 213.36 40.005 0)
 		(effects
 			(font
@@
 	)
 	(junction
-		(at 200.025 38.735)
-		(diameter 0)
-		(color 0 0 0 0)
-	)
-	(junction
 		(at 156.845 128.27)
 		(diameter 0)
@@
 		(color 0 0 0 0)
 	)
+	(junction
+		(at 200.025 38.735)
+		(diameter 0)
+		(color 0 0 0 0)
+	)
 	(bus
 		(pts
@@
 		)
 	)
-	(wire
-		(pts
-			(xy 200.025 38.735) (xy 215.265 38.735)
-		)
-		(stroke
-			(width 0)
-			(type default)
-		)
-	)
 	(bus
 		(pts
@@
 		)
 	)
-	(wire
-		(pts
-			(xy 215.265 48.26) (xy 215.265 38.735)
-		)
-		(stroke
-			(width 0)
-			(type default)
-		)
-	)
 	(bus
 		(pts
@@
 		)
 	)
+	(wire
+		(pts
+			(xy 215.265 45.72) (xy 215.265 48.26)
+		)
+		(stroke
+			(width 0)
+			(type default)
+		)
+	)
 	(bus
 		(pts
@@
 		)
 		(stroke
+			(width 0)
+			(type default)
+		)
+	)
+	(wire
+		(pts
+			(xy 200.025 38.735) (xy 205.105 38.735)
+		)
+		(stroke
